File: _autosave-TFG-PCB.kicad_pcb (KiCad board)
At the start: 2 copper layers, 141 parts, among them J1 TYPE-C-31-M-12, SW1 SW_Push, U1 ATmega32U4-AU, Y1 16MHz

Commit message: Renamed Footprints to account for keys
Parts:
- moved C3 0.13 mm to (226.2, 233.0)
Connections:
- J1 pad A5: Net-(J1-PadA5) -> CC1
- J1 pad B5: Net-(J1-PadB5) -> CC1
- R4 pad 2: Net-(J1-PadB5) -> CC1
Routing:
- net COL12: track 0.00 -> 89.5 mm
- net COL10: track 0.00 -> 88.1 mm
- net COL11: track 0.00 -> 87.6 mm
- net COL6: track 0.00 -> 87.6 mm
- net COL13: track 0.00 -> 83.6 mm
- net GND: track 0.00 -> 76.3 mm
- net COL7: track 0.00 -> 67.5 mm
- net COL8: track 0.00 -> 67.5 mm
- net COL9: track 0.00 -> 67.5 mm
- net COL2: track 23.0 -> 89.5 mm
- net COL3: track 23.0 -> 67.5 mm
- net COL4: track 23.0 -> 67.5 mm
- net COL5: track 23.0 -> 67.5 mm
- net +5V: track 0.00 -> 27.5 mm, vias 0 -> 3
- net Net-(C1-Pad1): track 0.00 -> 16.2 mm
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