File: _autosave-TFG-PCB.kicad_pcb (KiCad board)
At the start: 2 copper layers, 287.3 x 99.2 mm, 146 parts, among them J1 TYPE-C-31-M-12, SW1 SW_Push, U1 ATmega32U4-AU, Y1 16MHz

Commit message: Board created!
Included logo, fixed minor issues, generated board files + zipped gerbers into folder
Parts:
- moved G*** 4.40 mm to (264.0, 240.4)
Changed lines of the file:
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@@
   )
   (module "Logo lib:AM Logo 1.25in" (layer F.Cu)
-    (at 267.208 237.363)
+    (at 264.033 240.411)
     (fp_text reference G*** (at 0 0) (layer F.SilkS) hide
       (effects (font (size 1.524 1.524) (thickness 0.3)))
@@
       (xy -1.793673 -5.925123) (xy -1.447745 -6.064847) (xy -1.087967 -6.174745) (xy -0.713484 -6.255151)
       (xy -0.625997 -6.269384) (xy -0.456568 -6.289528) (xy -0.264677 -6.30245) (xy -0.060134 -6.30815)
-      (xy 0.147246 -6.306628)) (layer Eco2.User) (width 0.01))
+      (xy 0.147246 -6.306628)) (layer F.Cu) (width 0.01))
     (fp_poly (pts (xy 5.892666 3.863148) (xy 5.905044 3.873783) (xy 5.910451 3.900642) (xy 5.91176 3.951195)
       (xy 5.911784 3.96875) (xy 5.911104 4.026597) (xy 5.90691 4.059239) (xy 5.895979 4.074541)
       (xy 5.875084 4.080369) (xy 5.865527 4.081545) (xy 5.819269 4.086853) (xy 5.824186 3.974058)
       (xy 5.827509 3.914509) (xy 5.832944 3.880737) (xy 5.843479 3.865458) (xy 5.862099 3.861388)
-      (xy 5.870443 3.861263) (xy 5.892666 3.863148)) (layer Eco2.User) (width 0.01))
+      (xy 5.870443 3.861263) (xy 5.892666 3.863148)) (layer F.Cu) (width 0.01))
     (fp_poly (pts (xy 10.758413 4.597187) (xy 10.890821 4.597654) (xy 10.996675 4.599007) (xy 11.079232 4.601716)
       (xy 11.141752 4.606251) (xy 11.187494 4.613082) (xy 11.219718 4.622678) (xy 11.241681 4.63551)
@@
       (xy 11.051309 4.686562) (xy 10.97571 4.683067) (xy 10.876381 4.681037) (xy 10.750383 4.680085)
       (xy 10.594777 4.679822) (xy 10.563637 4.679818) (xy 10.004558 4.679818) (xy 10.004558 4.597135)
-      (xy 10.596191 4.597135) (xy 10.758413 4.597187)) (layer Eco2.User) (width 0.01))
+      (xy 10.596191 4.597135) (xy 10.758413 4.597187)) (layer F.Cu) (width 0.01))
     (fp_poly (pts (xy 9.234313 4.677271) (xy 9.362752 4.75165) (xy 9.466287 4.836189) (xy 9.472845 4.842669)
       (xy 9.524143 4.899533) (xy 9.571409 4.961782) (xy 9.611009 5.023263) (xy 9.639308 5.077825)
@@
       (xy 8.014877 5.31281) (xy 8.056481 5.157586) (xy 8.125989 5.013275) (xy 8.22168 4.883311)
       (xy 8.341833 4.771132) (xy 8.484727 4.680173) (xy 8.51064 4.667314) (xy 8.6403 4.605404)
-      (xy 9.089278 4.605404) (xy 9.234313 4.677271)) (layer Eco2.User) (width 0.01))
+      (xy 9.089278 4.605404) (xy 9.234313 4.677271)) (layer F.Cu) (width 0.01))
     (fp_poly (pts (xy 7.089387 4.605942) (xy 7.151185 4.6085) (xy 7.197257 4.61449) (xy 7.236272 4.625324)
       (xy 7.2769 4.642415) (xy 7.300847 4.653904) (xy 7.394533 4.712032) (xy 7.486163 4.790589)
@@
       (xy 6.625304 4.700331) (xy 6.705534 4.653904) (xy 6.750285 4.633106) (xy 6.789033 4.619281)
       (xy 6.830448 4.611015) (xy 6.883201 4.606896) (xy 6.955961 4.605512) (xy 7.003191 4.605404)
-      (xy 7.089387 4.605942)) (layer Eco2.User) (width 0.01))
+      (xy 7.089387 4.605942)) (layer F.Cu) (width 0.01))
     (fp_poly (pts (xy 5.866309 4.600171) (xy 5.911784 4.605404) (xy 5.911784 5.457031) (xy 5.911761 5.646497)
       (xy 5.911622 5.805566) (xy 5.911261 5.936914) (xy 5.910573 6.043216) (xy 5.909453 6.127148)
@@
       (xy 5.82623 6.164949) (xy 5.824524 6.066264) (xy 5.823091 5.947085) (xy 5.821973 5.810559)
       (xy 5.821214 5.659831) (xy 5.820857 5.498045) (xy 5.820834 5.444909) (xy 5.820834 4.594939)
-      (xy 5.866309 4.600171)) (layer Eco2.User) (width 0.01))
+      (xy 5.866309 4.600171)) (layer F.Cu) (width 0.01))
     (fp_poly (pts (xy 5.032922 3.860946) (xy 5.04552 3.872038) (xy 5.049732 3.894623) (xy 5.053469 3.945061)
       (xy 5.056528 4.018138) (xy 5.058709 4.108635) (xy 5.059812 4.211335) (xy 5.059904 4.245736)
@@
       (xy 4.968683 4.251047) (xy 4.969962 4.14467) (xy 4.971536 4.059476) (xy 4.973482 3.993086)
       (xy 4.975878 3.943122) (xy 4.978802 3.907207) (xy 4.982331 3.882962) (xy 4.986543 3.868009)
-      (xy 4.991517 3.859971) (xy 4.997329 3.856468) (xy 5.000298 3.855727) (xy 5.032922 3.860946)) (layer Eco2.User) (width 0.01))
+      (xy 4.991517 3.859971) (xy 4.997329 3.856468) (xy 5.000298 3.855727) (xy 5.032922 3.860946)) (layer F.Cu) (width 0.01))
     (fp_poly (pts (xy 4.709855 4.642611) (xy 4.706153 4.664205) (xy 4.696703 4.678083) (xy 4.674932 4.686598)
       (xy 4.634268 4.692102) (xy 4.568139 4.696947) (xy 4.555795 4.697751) (xy 4.444557 4.710708)
@@
       (xy 4.063244 4.852421) (xy 4.140686 4.766686) (xy 4.229486 4.692999) (xy 4.320208 4.640108)
       (xy 4.340869 4.63161) (xy 4.416436 4.60982) (xy 4.50231 4.59909) (xy 4.57405 4.597135)
-      (xy 4.715088 4.597135) (xy 4.709855 4.642611)) (layer Eco2.User) (width 0.01))
+      (xy 4.715088 4.597135) (xy 4.709855 4.642611)) (layer F.Cu) (width 0.01))
     (fp_poly (pts (xy 2.877544 4.60131) (xy 2.940639 4.610176) (xy 2.986207 4.621398) (xy 3.127692 4.677955)
       (xy 3.258943 4.760755) (xy 3.375366 4.864991) (xy 3.472365 4.985858) (xy 3.545347 5.118547)
@@
       (xy 2.246391 4.755502) (xy 2.377918 4.675746) (xy 2.439834 4.645747) (xy 2.48847 4.625789)
       (xy 2.534163 4.613467) (xy 2.587248 4.606372) (xy 2.658062 4.602098) (xy 2.701755 4.600328)
-      (xy 2.801166 4.598268) (xy 2.877544 4.60131)) (layer Eco2.User) (width 0.01))
+      (xy 2.801166 4.598268) (xy 2.877544 4.60131)) (layer F.Cu) (width 0.01))
     (fp_poly (pts (xy 0.971941 4.606042) (xy 1.034797 4.608834) (xy 1.081947 4.6151) (xy 1.12207 4.626155)
       (xy 1.163843 4.643319) (xy 1.178267 4.649984) (xy 1.297545 4.72277) (xy 1.40149 4.819525)
@@
       (xy 0.360284 4.838181) (xy 0.454161 4.74568) (xy 0.557318 4.671745) (xy 0.587939 4.655013)
       (xy 0.631971 4.633807) (xy 0.669778 4.619691) (xy 0.709945 4.611231) (xy 0.761057 4.606991)
-      (xy 0.8317 4.605537) (xy 0.884701 4.605404) (xy 0.971941 4.606042)) (layer Eco2.User) (width 0.01))
+      (xy 0.8317 4.605537) (xy 0.884701 4.605404) (xy 0.971941 4.606042)) (layer F.Cu) (width 0.01))
     (fp_poly (pts (xy -3.176274 4.605526) (xy -3.080957 4.606238) (xy -3.010744 4.608898) (xy -2.957684 4.614469)
       (xy -2.913823 4.623912) (xy -2.871209 4.638193) (xy -2.855445 4.64438) (xy -2.728577 4.710684)
@@
       (xy -3.910951 5.269832) (xy -3.933023 5.417439) (xy -4.028678 5.417439) (xy -4.023898 5.326019)
       (xy -3.985648 5.170798) (xy -3.919277 5.026007) (xy -3.826435 4.895099) (xy -3.708773 4.781529)
-      (xy -3.567941 4.688753) (xy -3.541868 4.675324) (xy -3.400792 4.605404) (xy -3.176274 4.605526)) (layer Eco2.User) (width 0.01))
+      (xy -3.567941 4.688753) (xy -3.541868 4.675324) (xy -3.400792 4.605404) (xy -3.176274 4.605526)) (layer F.Cu) (width 0.01))
     (fp_poly (pts (xy -4.275233 4.598092) (xy -4.223184 4.60494) (xy -4.193209 4.617177) (xy -4.189623 4.622151)
       (xy -4.188368 4.657493) (xy -4.216679 4.681315) (xy -4.275216 4.693961) (xy -4.331631 4.696354)
@@
       (xy -4.935725 5.051228) (xy -4.890344 4.933479) (xy -4.819547 4.824577) (xy -4.729242 4.730963)
       (xy -4.625334 4.659076) (xy -4.543717 4.623835) (xy -4.483598 4.609506) (xy -4.413462 4.600414)
-      (xy -4.341333 4.596596) (xy -4.275233 4.598092)) (layer Eco2.User) (width 0.01))
+      (xy -4.341333 4.596596) (xy -4.275233 4.598092)) (layer F.Cu) (width 0.01))
     (fp_poly (pts (xy -6.057336 4.600291) (xy -5.962447 4.61196) (xy -5.954576 4.613632) (xy -5.811105 4.661886)
       (xy -5.676111 4.738826) (xy -5.554182 4.840294) (xy -5.449909 4.962135) (xy -5.367882 5.100189)
@@
       (xy -6.969901 5.152331) (xy -6.964083 5.137477) (xy -6.898006 5.010796) (xy -6.806707 4.890631)
       (xy -6.697117 4.783894) (xy -6.576167 4.697498) (xy -6.471116 4.645799) (xy -6.38637 4.622079)
-      (xy -6.281214 4.606093) (xy -6.167564 4.598583) (xy -6.057336 4.600291)) (layer Eco2.User) (width 0.01))
+      (xy -6.281214 4.606093) (xy -6.167564 4.598583) (xy -6.057336 4.600291)) (layer F.Cu) (width 0.01))
     (fp_poly (pts (xy -7.19653 4.605452) (xy -7.183825 4.619276) (xy -7.187912 4.640173) (xy -7.204092 4.687794)
       (xy -7.230887 4.758701) (xy -7.266817 4.849459) (xy -7.310403 4.95663) (xy -7.360168 5.076778)
@@
       (xy -7.465847 5.069122) (xy -7.411833 4.945266) (xy -7.367299 4.844835) (xy -7.331135 4.765474)
       (xy -7.302227 4.70483) (xy -7.279464 4.660548) (xy -7.261733 4.630275) (xy -7.247922 4.611655)
-      (xy -7.236918 4.602334) (xy -7.230492 4.60011) (xy -7.19653 4.605452)) (layer Eco2.User) (width 0.01))
+      (xy -7.236918 4.602334) (xy -7.230492 4.60011) (xy -7.19653 4.605452)) (layer F.Cu) (width 0.01))
     (fp_poly (pts (xy -9.11202 3.85779) (xy -9.106951 3.863049) (xy -9.102609 3.873732) (xy -9.098939 3.892066)
       (xy -9.095884 3.92028) (xy -9.093388 3.960602) (xy -9.091395 4.015258) (xy -9.089849 4.086477)
@@
       (xy -9.17573 4.528992) (xy -9.17451 4.369387) (xy -9.173025 4.227237) (xy -9.171305 4.105213)
       (xy -9.169383 4.00599) (xy -9.167291 3.932241) (xy -9.16506 3.886641) (xy -9.163097 3.872038)
-      (xy -9.13693 3.856052) (xy -9.117875 3.855728) (xy -9.11202 3.85779)) (layer Eco2.User) (width 0.01))
+      (xy -9.13693 3.856052) (xy -9.117875 3.855728) (xy -9.11202 3.85779)) (layer F.Cu) (width 0.01))
     (fp_poly (pts (xy -10.067636 4.675324) (xy -9.928145 4.761196) (xy -9.807521 4.869363) (xy -9.709199 4.995378)
       (xy -9.636613 5.134792) (xy -9.593198 5.283157) (xy -9.591695 5.291667) (xy -9.585891 5.345632)
@@
       (xy -10.860209 4.697793) (xy -10.754059 4.64438) (xy -10.71004 4.628218) (xy -10.667503 4.617224)
       (xy -10.618496 4.610433) (xy -10.555064 4.606883) (xy -10.469256 4.605611) (xy -10.43323 4.605526)
-      (xy -10.208713 4.605404) (xy -10.067636 4.675324)) (layer Eco2.User) (width 0.01))
+      (xy -10.208713 4.605404) (xy -10.067636 4.675324)) (layer F.Cu) (width 0.01))
   )
   (module Resistor_SMD:R_0805_2012Metric (layer B.Cu)
