File: TFG-PCB.kicad_pcb (KiCad board)
At the start: 2 copper layers, 287.3 x 99.2 mm, 145 parts, among them J1 TYPE-C-31-M-12, SW1 SW_Push, U1 ATmega32U4-AU, Y1 16MHz

Commit message: PCB finished (almost)
PCB finished aside from ground fill and logo addition
Parts:
- moved C7 4.47 mm to (220.7, 247.5)
Connections:
- R1 pad 1: Net-(R1-Pad1) -> +5V
- U1 pad 18: Net-(U1-Pad18) -> COL6
- U1 pad 19: Net-(U1-Pad19) -> COL7
- U1 pad 20: Net-(U1-Pad20) -> COL8
- U1 pad 21: Net-(U1-Pad21) -> COL9
- U1 pad 22: Net-(U1-Pad22) -> COL10
- U1 pad 25: Net-(U1-Pad25) -> COL11
- U1 pad 26: Net-(U1-Pad26) -> COL12
- U1 pad 27: Net-(U1-Pad27) -> COL13
- U1 pad 28: Net-(U1-Pad28) -> ROW0
- U1 pad 29: Net-(U1-Pad29) -> ROW1
- U1 pad 30: Net-(U1-Pad30) -> ROW2
- U1 pad 31: Net-(U1-Pad31) -> ROW3
- U1 pad 32: Net-(U1-Pad32) -> ROW4
- U1 pad 36: Net-(U1-Pad36) -> COL0
- U1 pad 37: Net-(U1-Pad37) -> COL1
- U1 pad 38: Net-(U1-Pad38) -> COL2
- U1 pad 39: Net-(U1-Pad39) -> COL3
- U1 pad 40: Net-(U1-Pad40) -> COL4
- U1 pad 41: Net-(U1-Pad41) -> COL5
Routing:
- net COL13: track 82.3 -> 274.6 mm, vias 0 -> 1
- net COL12: track 90.0 -> 255.0 mm, vias 0 -> 1
- net ROW0: track 257.6 -> 411.4 mm, vias 2 -> 4
- net COL11: track 88.0 -> 228.2 mm, vias 0 -> 1
- net ROW1: track 263.5 -> 399.9 mm, vias 2 -> 4
- net ROW2: track 235.7 -> 353.6 mm, vias 2 -> 4
- net COL10: track 89.0 -> 201.8 mm, vias 0 -> 1
- net COL8: track 67.9 -> 170.8 mm, vias 0 -> 1
- net COL9: track 67.9 -> 170.8 mm, vias 0 -> 1
- net ROW3: track 247.3 -> 348.9 mm, vias 2 -> 4
- net COL0: track 83.0 -> 178.7 mm, vias 0 -> 1
- net COL1: track 87.6 -> 159.5 mm, vias 6 -> 7
- net COL7: track 67.9 -> 135.2 mm, vias 0 -> 1
- net RST: track 17.6 -> 81.3 mm, vias 0 -> 2
- net COL2: track 90.1 -> 137.8 mm, vias 2 -> 3
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